File: PCB/Marvelous65 Split.sch (KiCad schematic (older format))
At the start: 213 parts, among them J1 USB_C_Receptacle_USB2.0, J2 Conn_01x04, J3 AudioJack4, J4 Conn_01x02, J5 USB_C_Receptacle_USB2.0, J6 Conn_01x04, J7 AudioJack4, J8 Conn_01x02, SW1 SW_DPDT_x2, SW2 SW_PUSH, SW3 Rotary_Encoder_Switch, SW4 SW_PUSH, SW5 Rotary_Encoder_Switch, SW6 SW_DPDT_x2, U1 ProMicro, U2 USBLC6-2SC6, U3 ProMicro, U4 USBLC6-2SC6

Commit message: fix iso enter and panelization
Parts:
- ISO_ENTER1: footprint keyswitches:SW_MX -> MX_Only:MXOnly-ISO-ROTATED-ReversedStabilizers-NoLED
Changed lines of the file:
@@
 F 0 "ISO_ENTER1" H 8133 2073 60  0000 C CNN
 F 1 "MX-NoLED" H 8133 1999 20  0000 C CNN
-F 2 "keyswitches:SW_MX" H 7475 1825 60  0001 C CNN
+F 2 "MX_Only:MXOnly-ISO-ROTATED-ReversedStabilizers-NoLED" H 7475 1825 60  0001 C CNN
 F 3 "" H 7475 1825 60  0001 C CNN
 	1    8100 1850

Commit message: add a bunch of files
Parts:
- J1, J5: symbol Connector:USB_C_Receptacle_USB2.0 -> Marvelous65-Split-rescue:USB_C_Receptacle_USB2.0-Connector
- U2, U4: symbol Power_Protection:USBLC6-2SC6 -> Marvelous65-Split-rescue:USBLC6-2SC6-Power_Protection
Changed lines of the file:
@@
 $EndComp
 $Comp
-L Connector:USB_C_Receptacle_USB2.0 J1
+L Marvelous65-Split-rescue:USB_C_Receptacle_USB2.0-Connector J1
 U 1 1 5FF5FD4B
 P 1050 4650
@@
 $EndComp
 $Comp
-L Power_Protection:USBLC6-2SC6 U2
+L Marvelous65-Split-rescue:USBLC6-2SC6-Power_Protection U2
 U 1 1 5FF63170
 P 2850 6600
@@
 Connection ~ 21500 1700
 $Comp
-L Connector:USB_C_Receptacle_USB2.0 J5
+L Marvelous65-Split-rescue:USB_C_Receptacle_USB2.0-Connector J5
 U 1 1 6083EABF
 P 12950 4000
@@
 $EndComp
 $Comp
-L Power_Protection:USBLC6-2SC6 U4
+L Marvelous65-Split-rescue:USBLC6-2SC6-Power_Protection U4
 U 1 1 6087EFA5
 P 15100 3950
